File: hardware/pcb/Speaker.kicad_sch (KiCad schematic)
At the start: 6 parts, among them U5 MAX98357AETE+T

Commit message: Exclude unpopulated connectors from BOM
Parts:
- LS1: now left out of the parts list
Changed lines of the file:
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@@
   )
   (symbol (lib_id "Device:Speaker") (at 102.87 101.6 180) (unit 1)
-    (in_bom yes) (on_board yes) (dnp no) (fields_autoplaced)
+    (in_bom no) (on_board yes) (dnp no) (fields_autoplaced)
     (property "Reference" "LS1" (at 102.362 90.17 0)
       (effects (font (size 1.27 1.27)))
